File: test_board/test_board.kicad_pcb (KiCad board)
At the start: 4 copper layers, 100.9 x 88 mm, 167 parts, among them J3 Conn_01x02_Pin, SW1 CJS-1201B, U1 TLV3601DCKR, U10 TLV3601DCKR, U11 TLV3601DCKR, U12 TLV3601DCKR, U13 HC-PM254-8.5H-1X24PZ, U14 REF3012, U15 REF3025, U16 TLV75733PDBVR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

Commit message: added pcb
Parts:
- added C47: 10uF, PCM_JLCPCB:C_0805, F.Cu at (91.2, 87.0)
- R1, R11, R13, R15, R17, R19, R21, R23, R25, R27, R29, R3, R31, R33, R35, R37, R39, R5, R7, R9: value 1.5kΩ -> 3.3kΩ
Routing:
- net GND: track 41.6 -> 45.2 mm, vias 3933 -> 3936
- net +5V: track 6.58 -> 9.54 mm, vias 5 -> 6

Commit message: added 0 ohm resistor to comparator output
Parts:
- added R71: 0Ω, PCM_JLCPCB:R_0402, F.Cu at (79.2, 30.7)
- added R72: 0Ω, PCM_JLCPCB:R_0402, F.Cu at (79.2, 35.8)
- added R73: 0Ω, PCM_JLCPCB:R_0402, F.Cu at (79.2, 40.9)
- added R74: 0Ω, PCM_JLCPCB:R_0402, F.Cu at (79.2, 46.0)
- added R75: 0Ω, PCM_JLCPCB:R_0402, F.Cu at (79.2, 51.1)
- added R76: 0Ω, PCM_JLCPCB:R_0402, F.Cu at (79.2, 56.2)
- added R77: 0Ω, PCM_JLCPCB:R_0402, F.Cu at (79.2, 61.3)
- added R78: 0Ω, PCM_JLCPCB:R_0402, F.Cu at (79.2, 71.5)
- added R79: 0Ω, PCM_JLCPCB:R_0402, F.Cu at (79.2, 76.6)
- added R80: 0Ω, PCM_JLCPCB:R_0402, F.Cu at (79.2, 81.7)
- moved R59 0.47 mm to (79.2, 79.8)
- moved R57 0.45 mm to (79.2, 74.7)
- moved R55 0.43 mm to (79.2, 69.6)
- moved R53 0.27 mm to (79.2, 59.4)
- moved R51 0.26 mm to (79.2, 54.3)
- moved R41 0.26 mm to (79.2, 28.8)
- moved R42 0.26 mm to (79.2, 33.9)
- moved R45 0.26 mm to (79.2, 39.0)
- moved R47 0.26 mm to (79.2, 44.1)
- moved R49 0.26 mm to (79.2, 49.2)
Connections:
- U1 pad 1: in0 -> Net-(U1-OUT)
- U10 pad 1: in7 -> Net-(U10-OUT)
- U11 pad 1: in8 -> Net-(U11-OUT)
- U12 pad 1: in9 -> Net-(U12-OUT)
- U3 pad 1: in1 -> Net-(U3-OUT)
- U5 pad 1: in2 -> Net-(U5-OUT)
- U6 pad 1: in3 -> Net-(U6-OUT)
- U7 pad 1: in4 -> Net-(U7-OUT)
- U8 pad 1: in5 -> Net-(U8-OUT)
- U9 pad 1: in6 -> Net-(U9-OUT)
Routing:
- net Net-(U12-OUT): track 0.00 -> 1.21 mm
- net Net-(U11-OUT): track 0.00 -> 1.21 mm
- net Net-(U10-OUT): track 0.00 -> 1.21 mm
- net Net-(U8-OUT): track 0.00 -> 1.20 mm
- net Net-(U7-OUT): track 0.00 -> 1.20 mm
- net Net-(U6-OUT): track 0.00 -> 1.20 mm
- net Net-(U5-OUT): track 0.00 -> 1.20 mm
- net Net-(U3-OUT): track 0.00 -> 1.20 mm
- net Net-(U1-OUT): track 0.00 -> 1.20 mm
- net Net-(U9-OUT): track 0.00 -> 1.18 mm
- net in0: track 3.68 -> 2.95 mm
- net in1: track 3.68 -> 2.99 mm
- net in2: track 3.69 -> 3.02 mm
- net in3: track 3.70 -> 3.06 mm
- net in4: track 3.71 -> 3.10 mm
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