File: test_board/out.kicad_sch (KiCad schematic)
At the start: 3 parts

Commit message: fixed output
Parts:
- removed R1: 1.5kΩ, PCM_JLCPCB:R_0402, symbol PCM_JLCPCB-Resistors:0402,1.5kΩ
- added R1: 3.3kΩ, PCM_JLCPCB:R_0402, symbol PCM_JLCPCB-Resistors:0402,3.3kΩ
- R2: now not fitted; now left out of the parts list
Connections:
- net 3.3out: now also R1.1
- net 50m_out: now also R1.2
